File: KiCAD/SmallyMouse2.sch (KiCad schematic (older format))
At the start: 27 parts, among them IC1 AT90USB1287, J1 Exp Header, J2 Slow/Fast, J3 XCN1A, J4 JTAG, J5 Bootloader, J6 Reset, J7 EXT PWR, J8 A1200 PWR, P1 USB_A, Y1 16 MHz Crystal

Commit message: tweaks
Parts:
- removed J7: EXT PWR, Connector_PinHeader_2.54mm:PinHeader_1x02_P2.54mm_Vertical, symbol SmallyMouse2-rescue:CONN_01X02
- added D1: MBR120, Diode_SMD:D_SOD-123F, symbol Device:D_Schottky
- J8: value A1200 PWR -> PWR_SEL
Connections:
- net at J3.7 (Pin_7): now also D1.2 (A); no longer J8.1 (P1)
- new net: D1.1 (K), J8.1 (P1)
Other:
- moved on the sheet: J8
Changed lines of the file:
@@
 	8875 3200 9750 3200
 Wire Wire Line
-	9675 3000 9675 2775
+	9825 3000 9825 2775
 $Comp
 L power:+5V #PWR0101
 U 1 1 5DAEFDBF
-P 9675 2775
-F 0 "#PWR0101" H 9675 2625 50  0001 C CNN
-F 1 "+5V" H 9675 2915 50  0000 C CNN
-F 2 "" H 9675 2775 50  0000 C CNN
-F 3 "" H 9675 2775 50  0000 C CNN
-	1    9675 2775
+P 9825 2775
+F 0 "#PWR0101" H 9825 2625 50  0001 C CNN
+F 1 "+5V" H 9825 2915 50  0000 C CNN
+F 2 "" H 9825 2775 50  0000 C CNN
+F 3 "" H 9825 2775 50  0000 C CNN
+	1    9825 2775
 	1    0    0    -1
 $EndComp
@@
 $EndComp
 $Comp
-L SmallyMouse2-rescue:CONN_01X02 J7
-U 1 1 5E307571
-P 10050 1850
-F 0 "J7" H 10050 2000 50  0000 C CNN
-F 1 "EXT PWR" V 10150 1850 50  0000 C CNN
-F 2 "Connector_PinHeader_2.54mm:PinHeader_1x02_P2.54mm_Vertical" H 10050 1850 50  0001 C CNN
-F 3 "" H 10050 1850 50  0001 C CNN
-	1    10050 1850
-	1    0    0    1
-$EndComp
-Wire Wire Line
-	9675 1800 9675 1575
-$Comp
-L power:+5V #PWR0105
-U 1 1 5E30D7ED
-P 9675 1575
-F 0 "#PWR0105" H 9675 1425 50  0001 C CNN
-F 1 "+5V" H 9675 1715 50  0000 C CNN
-F 2 "" H 9675 1575 50  0000 C CNN
-F 3 "" H 9675 1575 50  0000 C CNN
-	1    9675 1575
-	1    0    0    -1
-$EndComp
-Wire Wire Line
-	9850 1800 9675 1800
-Wire Wire Line
-	9675 1900 9675 2150
-$Comp
-L power:GND #PWR0107
-U 1 1 5E31EEEF
-P 9675 2150
-F 0 "#PWR0107" H 9675 1900 50  0001 C CNN
-F 1 "GND" H 9675 2000 50  0000 C CNN
-F 2 "" H 9675 2150 50  0000 C CNN
-F 3 "" H 9675 2150 50  0000 C CNN
-	1    9675 2150
-	1    0    0    -1
-$EndComp
-Wire Wire Line
-	9850 1900 9675 1900
-$Comp
 L Device:CP_Small C11
 U 1 1 5E34F821
@@
 Connection ~ 5150 6975
 Wire Wire Line
-	9850 3000 9675 3000
-Wire Wire Line
-	8875 3100 9850 3100
+	10000 3000 9825 3000
 $Comp
 L SmallyMouse2-rescue:CONN_01X02 J8
 U 1 1 5E2D2C75
-P 10050 3050
-F 0 "J8" H 10050 3200 50  0000 C CNN
-F 1 "A1200 PWR" V 10150 3050 50  0000 C CNN
-F 2 "Connector_PinHeader_2.54mm:PinHeader_1x02_P2.54mm_Vertical" H 10050 3050 50  0001 C CNN
-F 3 "" H 10050 3050 50  0001 C CNN
-	1    10050 3050
+P 10200 3050
+F 0 "J8" H 10200 3200 50  0000 C CNN
+F 1 "PWR_SEL" V 10300 3050 50  0000 C CNN
+F 2 "Connector_PinHeader_2.54mm:PinHeader_1x02_P2.54mm_Vertical" H 10200 3050 50  0001 C CNN
+F 3 "" H 10200 3050 50  0001 C CNN
+	1    10200 3050
 	1    0    0    1
 $EndComp
@@
 	-1   0    0    1
 $EndComp
+$Comp
+L Device:D_Schottky D1
+U 1 1 5E4BB82E
+P 9825 3100
+F 0 "D1" H 9950 3050 50  0000 C CNN
+F 1 "MBR120" H 10050 3150 50  0000 C CNN
+F 2 "Diode_SMD:D_SOD-123F" H 9825 3100 50  0001 C CNN
+F 3 "~" H 9825 3100 50  0001 C CNN
+	1    9825 3100
+	-1   0    0    1
+$EndComp
+Wire Wire Line
+	9975 3100 10000 3100
+Wire Wire Line
+	9675 3100 8875 3100
 $EndSCHEMATC
